File: hw/pcb/cycloid.sch (KiCad schematic (older format))
At the start: 14 parts, among them J1 CONN_01X04_MALE, J10 CONN_01X03_MALE, J11 CONN_01X03_MALE, J2 CONN_01X04_MALE, J3 CONN_01X04_MALE, J4 CONN_01X04_MALE, J5 CONN_01X04_MALE, J6 CONN_01X04_MALE, J7 CONN_01X02_MALE, J8 CONN_01X03_MALE, J9 CONN_01X03_MALE, U1 Teensy3.2

Commit message: add schematic pdf
also make i2c pullups no-populate; we don't actually need or want them
Parts:
- R1, R2: value 4k7 -> N/P
Changed lines of the file:
@@
 LIBS:contrib
 LIBS:valves
-LIBS:teensy
 LIBS:cycloid-cache
 EELAYER 25 0
@@
 P 3600 1450
 F 0 "R1" V 3680 1450 50  0000 C CNN
-F 1 "4k7" V 3600 1450 50  0000 C CNN
+F 1 "N/P" V 3600 1450 50  0000 C CNN
 F 2 "Resistors_SMD:R_0805_HandSoldering" V 3530 1450 50  0001 C CNN
 F 3 "" H 3600 1450 50  0001 C CNN
@@
 P 3900 1450
 F 0 "R2" V 3980 1450 50  0000 C CNN
-F 1 "4k7" V 3900 1450 50  0000 C CNN
+F 1 "N/P" V 3900 1450 50  0000 C CNN
 F 2 "Resistors_SMD:R_0805_HandSoldering" V 3830 1450 50  0001 C CNN
 F 3 "" H 3900 1450 50  0001 C CNN
